Commit message: ALTERACOES

File: urdf/lophorina.urdf (robot description, URDF)
Before this commit: robot lophorina, 10 links, 9 joints
Links:
- link base_link: geometry collision box size=0.6 0.8 0.1; visual mesh filename=package://lophorina/meshes/robot_body.stl scale=0.001 0.001 0.001
Joints:
- joint motor_back_left_to_back_left_propeller: limit (none) -> effort=100 velocity=10000
- joint motor_back_right_to_back_right_propeller: limit (none) -> effort=100 velocity=10000
- joint motor_front_left_to_front_left_propeller: limit (none) -> effort=100 velocity=10000
- joint motor_front_right_to_front_right_propeller: limit (none) -> effort=100 velocity=10000
